File: fpga_blaster.kicad_sch (KiCad schematic)
At the start: 263 parts, among them J1 Conn_02x05_Odd_Even, J2 Conn_02x05_Odd_Even, J3 Conn_01x03, J4 Conn_02x05_Odd_Even, J5 HDMI_D_1.4, J8 HDMI_D_1.4, Q1 STR2P3LLH6(Pfet), Q2 2N3904, Q4 IPD60R145, Q6 IPD60R145, Q7 2N3906, Q9 2N3904, SW1 FIRE, SW2 SW_DIP_x03, SW3 ARM, U1 LT3420, U10 AMC3330, U11 TLV9102, U12 LTC6362, U13 TLV9102, U14 AMC3302, U15 LTC6362, U16 LTC6362, U17 AD7352, U18 IR2127, U19 S80KS2563GABHV020, U2 MAX10, U20 TLV74318, U21 LM809, U22 MAX3227, U3 AD7352, U4 TLV74325, U5 4940, U6 4945, U7 LTC6362, U8 AMC3330, U9 AMC3302, X1 ASE-48MHz

Commit message: PCB V0.8 tapeout
Parts:
- removed L1: 600uH 0.5A, Inductor_SMD:L_2010_5025Metric, symbol Device:L_Ferrite
- removed Q7: 2N3906, Package_TO_SOT_SMD:SOT-23, symbol Transistor_BJT:2N3906
- removed Q9: 2N3904, Package_TO_SOT_SMD:SOT-23, symbol Transistor_BJT:2N3904
- removed U11, U13: TLV9102, Package_TO_SOT_SMD:SOT-23-5, symbol Amplifier_Operational:TLV9062
- added C100, C101, C102, C103, C104, C105, C106, C107, C108, C109, C110, C111, C112, C113, C114, C115, C116, C117, C118, C119, C120, C121, C122, C123, C124, C125, C126, C127, C131, C97, C98, C99: 0.1u, Capacitor_SMD:C_0603_1608Metric, symbol Device:C_Small
- added C128, C129, C130: 1u, Capacitor_SMD:C_0603_1608Metric, symbol Device:C_Small
- added C132, C133, C134, C135, C136, C137: 4.7u, Capacitor_SMD:C_1206_3216Metric, symbol Device:C_Small
- added D19: BAV99, Package_TO_SOT_SMD:SOT-23, symbol Diode:1N4007
- added D20: CRC_ERR, LED_SMD:LED_0603_1608Metric, symbol Device:LED
- added FB10, FB11, FB8, FB9: Ferrite, Inductor_SMD:L_0603_1608Metric, symbol Device:FerriteBead_Small
- added H1, H10, H11, H12, H13, H14, H15, H2, H3, H4, H5, H6, H7, H8, H9: ~, MountingHole:MountingHole_3mm_Pad, symbol Mechanical:MountingHole_Pad
- added J10, J11, J12, J13, J7, J9: Screw_Terminal_01x02, TerminalBlock_Phoenix:TerminalBlock_Phoenix_MKDS-1,5-2-5.08_1x02_P5.08mm_Horizontal, symbol Connector:Screw_Terminal_01x02
- added J6: Conn_02x05_Odd_Even, Connector_PinHeader_2.54mm:PinHeader_2x05_P2.54mm_Vertical, symbol Connector_Generic:Conn_02x05_Odd_Even
- added Q3: 2N3906, Package_TO_SOT_SMD:SOT-23, symbol Transistor_BJT:2N3906
- added Q5, Q7, Q8: 2N3904, Package_TO_SOT_SMD:SOT-23, symbol Transistor_BJT:2N3904
- added R100, R101, R103, R104, R110, R99: 0R, Resistor_SMD:R_0603_1608Metric, symbol Device:R
- added R102: 0.005R 1W, myspace pcb:R_2818 current sense, symbol Device:R
- added R105, R106, R107: 22R, Resistor_SMD:R_0603_1608Metric, symbol Device:R
- added R108, R109, R111: 1K, Resistor_SMD:R_0603_1608Metric, symbol Device:R
- added R112: DNI, Resistor_SMD:R_0603_1608Metric, symbol Device:R
- added R98: 10K, Resistor_SMD:R_0603_1608Metric, symbol Device:R
- added SW4, SW7, SW8: ARM, myspace pcb:SW_SPST_HP03, symbol Switch:SW_Push
- added SW5, SW6, SW9: FIRE, myspace pcb:SW_SPST_HP03, symbol Switch:SW_Push
- added TP1, TP2, TP3, TP4, TP7: ~, TestPoint:TestPoint_Keystone_5000-5004_Miniature, symbol Connector:TestPoint
- added U11, U13: TLV9062xD, Package_TO_SOT_SMD:SOT-23-8, symbol Amplifier_Operational:TLV9062xD
- added U23: TLV74325, Package_TO_SOT_SMD:SOT-23-5, symbol myspace:TLV74325_SOT23-5
- BT1: value 2462 -> ~
- C1, C10, C11, C18, C20, C26, C3, C30, C34, C45, C5, C50, C51, C66, C7, C70, C75, C87, C88, C89, C90, C91: DPN (none) -> 399-C0603C105K3RAC7867CT-ND
- C12, C21, C59, C61, C63, C8: DPN (none) -> 399-C1206C106K4PAC7800CT-ND
- C13, C14, C22, C24, C25, C42, C43, C58, C60, C62, C64, C68, C83, C84, C9, C92, C93, C94, C95, C96: DPN (none) -> 399-C0603C104K3RAC7867CT-ND
- C15: DPN (none) -> 399-13296-1-ND
- C16, C19: DPN (none) -> 399-C1206C475K5PAC7800CT-ND
- C17: footprint Capacitor_THT:C_Radial_D6.3mm_H5.0mm_P2.50mm -> Capacitor_THT:C_Radial_D5.0mm_H7.0mm_P2.00mm; DPN (none) -> 1572-1659-ND
- C2: value 0.1u -> 0.001u; DPN (none) -> 399-C0603C102K3RAC7867CT-ND
- C23, C28, C31, C37, C38, C39, C40, C41, C47, C48, C52, C54, C55, C56, C57, C71, C74, C77, C78, C80: value 1n -> 0.001u; DPN (none) -> 399-C0603C102K3RAC7867CT-ND
- C27, C36, C44, C72: value 10n -> 0.01u; DPN (none) -> 399-C0603C103K3RAC7867CT-ND
- C29, C32, C35, C46, C49, C53, C69, C73, C76, C79, C81, C82: value 100n -> 0.1u; DPN (none) -> 399-C0603C104K3RAC7867CT-ND
- C33, C4, C6, C65: DPN (none) -> 399-C0603C103K3RAC7867CT-ND
- C67: DPN (none) -> 1572-1041-ND
- C85: value 1u -> 0.1u; DPN (none) -> 399-C0603C104K3RAC7867CT-ND
- C86: value 1n -> 0.1u; DPN (none) -> 399-C0603C104K3RAC7867CT-ND
- D1, D13, D14, D15, D16, D2, D4, D6, D8: DPN (none) -> 754-2039-1-ND
- D10, D9: footprint Package_TO_SOT_SMD:TO-252-2 -> Package_TO_SOT_SMD:TO-263-2_TabPin1; DPN (none) -> 497-STPSC10065G2-TRCT-ND
- D11, D12: value SBYV26C -> ES1J; DPN (none) -> 1655-ES1JCT-ND
- D17: value STS -> nSTATUS; DPN (none) -> 754-2039-1-ND
- D18: value CONF -> CONF_DONE; DPN (none) -> 754-2039-1-ND
- D3: value 1N4001 -> BAV99; DPN (none) -> 1655-BAV99CT-ND
- D5: value MMBD3004SE -> GSD2004S; DPN (none) -> GSD2004S-E3-08CT-N
- D7: value FIRE -> CONTINUITY; DPN (none) -> 754-2039-1-ND
- FB1, FB2, FB3, FB4, FB5, FB6, FB7: DPN (none) -> 490-5254-1-ND
- J1, J2, J4: DPN (none) -> 732-2672-ND
- J3: DPN (none) -> 732-5316-ND
- J5, J8: footprint Connector_HDMI:HDMI_Micro-D_Molex_46765-0x01 -> Connector_HDMI:HDMI_A_Amphenol_10029449-x01xLF_Horizontal; symbol Connector:HDMI_D_1.4 -> Connector:HDMI_A; DPN (none) -> 609-4614-1-ND
- L2: DPN (none) -> M8893-ND
- LS1: DPN (none) -> 668-1068-1-ND
- Q4, Q6: DPN (none) -> 448-IPD60R145CFD7ATMA1CT-ND; OK (none) -> OK
- R1, R10, R11, R6, R7, R71, R72, R75, R76, R77, R95: DPN (none) -> P10.0KHCT-ND
- R12, R74: value 1K -> 22R; DPN (none) -> P22.0HCT-ND
- R13, R14, R15, R31, R4: DPN (none) -> P0.0GCT-ND
- R16, R17, R18, R19, R67, R68, R69, R70: DPN (none) -> P22.0HCT-ND
- R2, R23, R32: DPN (none) -> P100KHCT-ND
- R20, R21, R80, R81: DPN (none) -> 541-MCT0603MD2004BP500CT-ND
- R22: value 2R -> 10R; DPN (none) -> P10.0HCT-ND
- R24, R51: DPN (none) -> P0.0GCT-ND; JLC C491211 -> C778416
- R25, R26, R33, R34: DPN (none) -> P10.0HCT-ND
- R27, R30, R52, R79: DPN (none) -> P47KGCT-ND
- R28, R82: DPN (none) -> 10-ERA-3VRW1002VCT-ND
- R29: DPN (none) -> P51.1KDBCT-ND
- R34: footprint Package_TO_SOT_SMD:TO-252-2 -> Package_TO_SOT_SMD:TO-263-2_TabPin1; DPN 118-PWR163S-25-3301J-ND -> 118-PWR263S-20-3301F-ND; OK (none) -> OK
- R35, R36, R41, R42, R53, R54, R55, R56: DPN (none) -> P1.5KDBCT-ND
- R37, R38, R43, R44, R57, R58, R59, R60: DPN (none) -> P3.01KDBCT-ND
- R39, R40, R45, R46, R61, R62, R63, R64: value 30R -> 22R; DPN (none) -> P22.0HCT-ND
- R47, R48, R65, R66: value 10.0K -> 10.01K; DPN (none) -> 10-ERA-3VRW1002VCT-ND
- R49: value 0.005R 1W -> 0R; footprint Package_TO_SOT_SMD:TO-252-2 -> Resistor_SMD:R_0603_1608Metric; DPN (none) -> P0.0GCT-ND; JLC C723574 -> C778416
- R5, R73, R78, R83, R84, R85, R86, R87, R88, R89, R9, R90, R91, R92: DPN (none) -> P1.00KHCT-ND
- R50: footprint Package_TO_SOT_SMD:TO-252-2 -> myspace pcb:R_2818 current sense; DPN (none) -> 541-3275-1-ND; JLC C723574 -> (none); OK (none) -> OK
- R8: DPN (none) -> P2.00KHCT-ND
- SW1, SW3: footprint Button_Switch_SMD:SW_Push_1P1T_NO_CK_KSC6xxJ -> myspace pcb:SW_SPST_HP03; DPN (none) -> 360-2595-1-ND
- SW2: DPN (none) -> CT2193LPST-ND
- TP5: value 3V -> ~; footprint TestPoint:TestPoint_THTPad_D1.5mm_Drill0.7mm -> TestPoint:TestPoint_Keystone_5000-5004_Miniature; DPN (none) -> 36-1037-ND
- TP6: value GND -> ~; footprint TestPoint:TestPoint_THTPad_D1.5mm_Drill0.7mm -> TestPoint:TestPoint_Keystone_5000-5004_Miniature; DPN (none) -> 36-1037-ND
- TR1: footprint RF_Mini-Circuits:Mini-Circuits_CD542_H2.84mm -> myspace pcb:PA0637A Pulse Coil; DPN (none) -> 553-1978-1-ND
- U1: DPN (none) -> LT3420EMS#PBF-ND
- U10, U8: DPN (none) -> 296-AMC3330QDWERQ1CT-ND
- U12, U15, U16, U7: footprint Package_DFN_QFN:DFN-8-1EP_3x3mm_P0.5mm_EP1.66x2.38mm -> Package_SO:MSOP-8_3x3mm_P0.65mm; symbol Amplifier_Operational:LTC6362xDD -> Amplifier_Operational:LTC6362xMS8; DPN (none) -> 505-LTC6362CMS8#PBF-ND
- U14, U9: DPN (none) -> 296-AMC3302DWERCT-ND
- U17, U3: footprint Package_SO:TSSOP-16-1EP_4.4x5mm_P0.65mm_EP3x3mm_ThermalVias -> Package_SO:TSSOP-16_4.4x5mm_P0.65mm; DPN (none) -> 505-AD7352BRUZ-ND
- U18: DPN (none) -> IR2127SPBFCT-ND
- U19: footprint Package_BGA:BGA-25_6.35x6.35mm_Layout5x5_P1.27mm -> myspace pcb:FBGA-24_6mmx8mm_Layout5x5_P1.00mm; DPN (none) -> 448-S80KS2563GABHV020-ND
- U2: value MAX10 -> MAX10M04; DPN 544-3098-ND -> 544-3054-ND
- U20: DPN (none) -> 296-48712-1-ND
- U21: DPN (none) -> LM809M3-2.63/NOPBCT-ND
- U22: DPN (none) -> 296-19849-1-ND
- U4: DPN (none) -> 296-48989-1-ND
- U5: value 4940 -> LMO78_03-1.0; DPN (none) -> 3182-LMO78_03-1.0-ND
- U6: DPN (none) -> 2183-4945-ND
- X1: footprint Oscillator:Oscillator_SMD_Abracon_ASE-4Pin_3.2x2.5mm -> Oscillator:Oscillator_SMD_Abracon_ASV-4Pin_7.0x5.1mm_HandSoldering; DPN (none) -> 535-9328-1-ND
Connections:
- net dataa0 is gone; now on net dataA0: R18.1
- net dataa1 is gone; now on net dataA1: R69.1
- net datab0 is gone; now on net dataB0: R19.1
- net datab1 is gone; now on net dataB1: R70.1
- net +12V: now also C33.1, C66.1, U5.1 (VI), Q3.1 (E)
- net +1V8: now also U19.B1 (nCK), C119.1, C97.1
- net +2V5: now also C129.1, U23.5 (OUT); no longer C14.1, C24.1, C25.1, C43.1, U12.3 (V+), U12.7 (~{SHDN}), U15.3 (V+), U15.7 (~{SHDN}), U16.3 (V+), U16.7 (~{SHDN}), U7.3 (V+), U7.7 (~{SHDN})
- net +3.3V: now also C14.1, C24.1, C25.1, C43.1, LS1.1, U12.3 (V+), U12.7 (~{SHDN}), U15.3 (V+), U15.7 (~{SHDN}), U16.3 (V+), U16.7 (~{SHDN}), U7.3 (V+), U7.7 (~{SHDN}), C100.1, C101.1, C102.1, C103.1, C104.1, C105.1, C106.1, C107.1, C116.1, C117.1, C118.1, C121.1, C122.1, C123.1, C124.1, C125.1, C126.1, C127.1, C128.1, C131.1, C132.1, C133.1, C134.1, C135.1, C136.1, C137.1, C98.1, C99.1, D19.1 (K), FB10.1, FB11.1, FB8.1, FB9.1, J6.2 (Pin_2), R109.2, R98.1, SW5.2, SW6.2, SW9.2, U11.8 (V+), U13.8 (V+), U23.1 (IN)
- net +3.3VA: now also C108.1, C109.1, C110.1, C111.1, C112.1, C113.1, C130.1, FB10.2, FB11.2, FB8.2, FB9.2
- net +300V: now also R100.1; no longer FB2.2, FB3.2
- net +BATT: now also J12.2 (Pin_2), J9.2 (Pin_2), SW4.2, SW7.2, SW8.2; no longer C33.1, C66.1, TP5.1, U5.1 (VI)
- net CIdiag: now also U2.96 (IO); no longer U2.105 (IO)
- net CIhi: now also R101.2; no longer C67.1, R20.1, R50.1
- net CVdiag: now also U2.97 (VREFB6N); no longer U2.106 (IO)
- net GND: now also J2.10 (Pin_10), J2.3 (Pin_3), J5.11 (CKS), J5.17 (GND), J5.2 (D2S), J5.5 (D1S), J5.8 (D0S), J5.SH, J8.11 (CKS), J8.17 (GND), J8.2 (D2S), J8.5 (D1S), J8.8 (D0S), J8.SH, TP5.1, C100.2, C101.2, C102.2, C103.2, C104.2, C105.2, C106.2, C107.2, C108.2, C109.2, C110.2, C111.2, C112.2, C113.2, C114.2, C115.2, C116.2, C117.2, C118.2, C119.2, C120.2, C121.2, C122.2, C123.2, C124.2, C125.2, C126.2, C127.2, C128.2, C129.2, C130.2, C131.2, C132.2, C133.2, C134.2, C135.2, C136.2, C137.2, C97.2, C98.2, C99.2, H4.1, H5.1, H6.1, H7.1, J10.2 (Pin_2), J13.2 (Pin_2), J6.10 (Pin_10), J7.2 (Pin_2), J9.1 (Pin_1), Q5.1 (E), Q7.1 (E), Q8.1 (E), R104.2, TP1.1, TP2.1, TP3.1, TP4.1, U11.4 (V-), U13.4 (V-), U23.2 (GND); no longer C2.2, J2.4 (Pin_4), J2.5 (Pin_5), J5.16 (GND), J8.16 (GND), R21.1, R24.2, R81.1, U12.9 (V-), U15.9 (V-), U16.9 (V-), U7.9 (V-)
- net LIdiag: now also U2.93 (IO); no longer U2.101 (IO)
- net LIhi: no longer D10.1 (A), L2.2
- net LVdiag: now also U2.98 (IO); no longer U2.102 (IO)
- net ain_1: now also U2.14 (ADC1IN8); no longer U2.6 (ADC1IN1)
- net ain_2: now also U2.13 (ADC1IN7); no longer U2.7 (ADC1IN2)
- net ain_3: now also J4.4 (Pin_4), U2.12 (ADC1IN6); no longer J4.5 (Pin_5), U2.8 (ADC1IN3)
- net ain_4: now also J4.5 (Pin_5), U2.11 (ADC1IN5); no longer J4.7 (Pin_7), U2.10 (ADC1IN4)
- net ain_5: now also J4.6 (Pin_6), U2.10 (ADC1IN4); no longer J4.4 (Pin_4), U2.11 (ADC1IN5)
- net ain_6: now also J4.7 (Pin_7), U2.8 (ADC1IN3); no longer J4.6 (Pin_6), U2.12 (ADC1IN6)
- net ain_7: now also U2.7 (ADC1IN2); no longer U2.13 (ADC1IN7)
- net ain_8: now also U2.6 (ADC1IN1); no longer U2.14 (ADC1IN8)
- net arm: now also J6.9 (Pin_9)
- net arm_led: now also J6.6 (Pin_6)
- net charge: now also U2.62 (IO); no longer U2.69 (IO)
- net conf_done: now also J6.4 (Pin_4)
- net cont_led: now also J6.3 (Pin_3)
- net cont_n: now also U2.69 (IO), Q5.3 (C); no longer U2.66 (IO)
- net cs: now also U2.106 (IO); no longer U2.92 (IO)
- net dataA0: now also U2.99 (IO); no longer U2.91 (IO)
- net dataA1: now also U2.102 (IO); no longer U2.90 (IO)
- net dataB0: now also U2.100 (IO); no longer U2.88 (IO)
- net dataB1: now also U2.105 (IO); no longer U2.89 (IO)
- net devclrn: now also R112.2
- net done: now also U2.64 (IO); no longer U2.70 (IO)
- net dump: now also U2.66 (IO); no longer U2.64 (IO)
- net fire: now also J6.1 (Pin_1), R107.2, SW5.1, SW6.1, SW9.1; no longer U2.124 (IO)
- net gate: now also Q4.1 (G), R22.2; no longer R22.1, U18.7 (HO)
- net hdmi2_ck+: now also J5.10 (CK+), U2.52 (IO); no longer J5.12 (CK+), U2.60 (IO)
- net hdmi2_ck-: now also J5.12 (CK-), U2.50 (IO); no longer J5.14 (CK-), U2.59 (IO)
- net hdmi2_d0+: now also J5.7 (D0+), U2.56 (IO); no longer J5.9 (D0+), U2.52 (IO)
- net hdmi2_d0-: now also J5.9 (D0-), U2.55 (IO); no longer J5.11 (D0-), U2.50 (IO)
- net hdmi2_d1+: now also J5.4 (D1+), U2.58 (IO); no longer J5.6 (D1+), U2.56 (IO)
- net hdmi2_d1-: now also J5.6 (D1-), U2.57 (IO); no longer J5.8 (D1-), U2.55 (IO)
- net hdmi2_d2+: now also J5.1 (D2+), U2.60 (IO); no longer J5.3 (D2+), U2.58 (IO)
- net hdmi2_d2-: now also J5.3 (D2-), U2.59 (IO); no longer J5.5 (D2-), U2.57 (IO)
- net hdmi_ck+: now also J8.10 (CK+), U2.39 (IO); no longer J8.12 (CK+), U2.47 (IO)
- net hdmi_ck-: now also J8.12 (CK-), U2.38 (IO); no longer J8.14 (CK-), U2.46 (IO)
- net hdmi_d0+: now also J8.7 (D0+), U2.43 (IO); no longer J8.9 (D0+), U2.39 (IO)
- net hdmi_d0-: now also J8.9 (D0-), U2.41 (IO); no longer J8.11 (D0-), U2.38 (IO)
- net hdmi_d1+: now also J8.4 (D1+), U2.45 (IO); no longer J8.6 (D1+), U2.43 (IO)
- net hdmi_d1-: now also J8.6 (D1-), U2.44 (IO); no longer J8.8 (D1-), U2.41 (IO)
- net hdmi_d2+: now also J8.1 (D2+), U2.47 (IO); no longer J8.3 (D2+), U2.45 (IO)
- net hdmi_d2-: now also J8.3 (D2-), U2.46 (IO); no longer J8.5 (D2-), U2.44 (IO)
- net iset0: now also J6.7 (Pin_7)
- net iset1: now also J6.8 (Pin_8)
- net iset2: now also J6.5 (Pin_5)
- net pwm: now also R105.1; no longer U18.2 (IN)
- net reset_n: now also R112.1
- net rx: now also U2.24 (IO), R106.2; no longer U2.21 (IO), U22.9 (R1OUT)
- net rx232: now also J3.1 (Pin_1); no longer J3.2 (Pin_2)
- net sclk: now also U2.101 (IO); no longer U2.93 (IO)
- net spi_clk: now also U2.87 (IO); no longer U2.85 (IO)
- net spi_cs: now also U2.81 (IO); no longer U2.78 (IO)
- net spi_d0: now also U2.78 (IO); no longer U2.75 (IO)
- net spi_d1: now also U2.85 (IO); no longer U2.74 (IO)
- net spi_d2: now also U2.75 (IO); no longer U2.79 (IO)
- net spi_d3: now also U2.77 (IO); no longer U2.81 (IO)
- net spi_d4: now also U2.76 (IO); no longer U2.86 (IO)
- net spi_d5: now also U2.79 (IO); no longer U2.84 (IO)
- net spi_d6: now also U2.84 (IO); no longer U2.76 (IO)
- net spi_d7: now also U2.86 (IO); no longer U2.77 (IO)
- net spi_ds: now also U2.74 (IO); no longer U2.87 (IO)
- net spk+: now also R108.1; no longer LS1.1
- net spk-: no longer LS1.2
- net tdi: no longer R77.2
- net tms: now also R77.2
- net tx: now also U2.25 (IO); no longer U2.22 (IO)
- net tx232: now also J3.2 (Pin_2); no longer J3.1 (Pin_1)
- net vina0+: now also C38.1, R39.2; no longer C40.1, R45.2
- net vina0-: now also C39.1, R40.2; no longer C41.1, R46.2
- net vinb0+: now also C40.1, R45.2; no longer C38.1, R39.2
- net vinb0-: now also C41.1, R46.2; no longer C39.1, R40.2
- net HGNDLV: now reaches C72.2, C75.2, C76.1, C77.2, C78.2, C79.2, R81.2, R82.1, U8.2 (DCDC_HGND), U8.7 (INN), U8.8 (HGND)
- net at U16.2 (VOCM): now also U13.6 (-), U13.7; no longer U15.2 (VOCM)
- net SW: now reaches TR1.2
- net SW: now also R29.2, U1.6 (SW)
- net at R23.1: now also Q3.2 (B)
- net at R71.2: now also Q3.3 (C)
- net HGNDLI: now reaches C45.2, C46.1, C47.2, C48.2, C49.2, FB7.1, U14.2 (DCDC_HGND), U14.8 (HGND)
- net ANAIN1: now reaches C2.1, R4.1, U2.3 (ANAIN1)
- net ANAIN1: now also TP7.1
- net REFGND: now reaches FB1.1, U2.4 (REFGDN)
- net REFGND: now also C2.2
- net CIoutp: now reaches R41.1, U9.11 (OUTP)
- net dio0: now reaches J2.1 (Pin_1)
- net dio0: now also U2.118 (IO); no longer U2.110 (IO)
- net dio4: now reaches U2.111 (IO)
- net dio4: now also J2.7 (Pin_7); no longer J2.3 (Pin_3)
- net dio5: now reaches U2.112 (VREFB7N)
- net dio5: now also J2.8 (Pin_8); no longer J2.9 (Pin_9)
- net dio2: now reaches U2.113 (IO)
- net dio2: now also J2.5 (Pin_5); no longer J2.7 (Pin_7)
- net dio1: now reaches J2.2 (Pin_2)
- net dio1: now also U2.119 (IO); no longer U2.114 (IO)
- net vccio7: now reaches C90.1, R31.2, U2.117 (VCCIO7)
- net vccio7: now also J2.4 (Pin_4), C120.1; no longer J2.10 (Pin_10)
- net dio3: now reaches J2.6 (Pin_6)
- net dio3: now also U2.114 (IO); no longer U2.118 (IO)
- net HGNDCV: now reaches C36.2, C50.2, C73.1, C74.2, C80.2, C81.2, R21.2, R28.1, U10.2 (DCDC_HGND), U10.7 (INN), U10.8 (HGND)
- net CVoutn: now reaches U10.10 (OUTN)
- net CVoutn: now also R54.1; no longer R35.1
- net LVoutp: now reaches R55.1, U8.11 (OUTP)
- net LIoutn: now reaches U14.10 (OUTN)
- net LIoutn: now also R35.1; no longer R54.1
- net VCCIO1B: now reaches C89.1, J1.4 (Pin_4), R14.2, R75.1, R76.1, R77.1, U2.23 (VCCIO1B)
- net VCCIO1B: now also C115.1
- net CVoutp: now reaches U10.11 (OUTP)
- net CVoutp: now also R53.1; no longer R36.1
- net at C42.1, R47.1, R48.2: now also U11.3 (+), U11.5 (+)
- net LVoutn: now reaches R56.1, U8.10 (OUTN)
- net HGNDCI: now reaches C28.2, C29.2, C30.2, C31.2, C32.1, FB2.1, U9.2 (DCDC_HGND), U9.8 (HGND)
- net +VSW: now reaches C84.2, D9.2 (K), Q4.3 (S), U18.5 (VS), U18.6 (CS)
- net +VSW: now also R49.1, R102.2; no longer L2.1
- net LVhi: now reaches R24.1
- net LVhi: now also R80.1; no longer J8.SH
- net SWDIS: now reaches Q6.2 (D), R34.1
- net VCCIO1A: now reaches C91.1, J4.2 (Pin_2), R15.2, U2.9 (VCCIO1A)
- net VCCIO1A: now also C114.1
- net B+: now reaches BT1.1 (+), SW3.1
- net B+: now also J12.1 (Pin_1), SW4.1, SW7.1, SW8.1
- net LIoutp: now reaches U14.11 (OUTP)
- net LIoutp: now also R36.1; no longer R53.1
- net crc: now reaches U2.134 (CRC_ERR)
- net crc: now also R111.2
- net at Q1.3 (D), R2.2: now also R110.1; no longer Q6.1 (G)
- net at C58.1, R65.1, R66.2: now also U13.3 (+), U13.5 (+)
- net CVlo: now reaches R51.1
- net CVlo: now also R21.1; no longer J5.SH
- net at U12.2 (VOCM): now also U11.1, U11.2 (-); no longer U7.2 (VOCM)
- net at R71.1: now also Q5.2 (B)
- net spi_nrst: now reaches U2.80 (VREFB5N)
- net spi_nrst: now also U19.A4 (nRST)
- net CIoutn: now reaches R42.1, U9.10 (OUTN)
- removed net IGNITER+: D11.1 (K), FB6.2, FB7.2, R49.1, R80.1
- new net: D19.2 (A), LS1.2, Q7.3 (C)
- new net: U13.1, U13.2 (-), U15.2 (VOCM)
- new net: Q7.2 (B), R108.2
- new net: D20.2 (A), R109.1
- new net: R22.1, U18.7 (HO)
- new net: Q8.2 (B), R111.1
- new net: R107.1, U2.124 (IO)
- new net: R106.1, U22.9 (R1OUT)
- new net: D20.1 (K), Q8.3 (C)
- new net: U11.6 (-), U11.7, U7.2 (VOCM)
- new net: R98.2, U23.3 (EN)
- new net +OUT: D10.1 (A), D11.1 (K), J11.1 (Pin_1), J13.1 (Pin_1), J7.1 (Pin_1), L2.2, R24.2
- new net CIlo: FB2.2, FB3.2, R100.2
- new net CSEN: C67.1, J10.1 (Pin_1), R101.1, R50.1, R99.2
- new net CVhi: R20.1, R99.1
- new net DisG: Q6.1 (G), R110.2
- new net LIlo: FB6.2, FB7.2, R103.2
- new net LSEN: J11.2 (Pin_2), L2.1, R102.1, R103.1
- new net LVlo: R104.1, R81.1
- new net dio6: J2.9 (Pin_9), U2.110 (IO)
- new net pwmr: R105.2, U18.2 (IN)
- no-connect marks 19 -> 31
Other:
- note added: "1x gain pre-amps"
- note added: "2.0x gain"
- note added: "41x gain"
- note added: "Current Probes"
- note added: "Front Panel extension"
- note added: "Igniter"
- note added: "Ishunt"
- note added: "Sampling ADCs simultaneous 4ch 12bit 3mhz isolated zero latency"
- note added: "ToDo: X - Add well placed buttons N - ADC in battery voltage (do externally), add VIN0? X - Fixup Amp Polarities and gain. - Calc all resistor values N - Split into Sheets/Zones X - Finalize Parts Lists (DK and JLC) X - Add Decoupling everywhere - Add Test points and ground clips - more LED Outputs (inc FPGA config) - I/O Connectors maximize"
- note added: "Voltage Probes"
- note removed: "Ignitor Energy"
- note removed: "Sampling ADCs"
- note removed: "ToDo: -Split into Sheets -Finalize Parts Lists (DK and JLC) -Add Decoupling everywhere -Add Test points and ground clips (Logic Analyser output) -Amp Polarities and Resistor Values -more LED Outputs (inc FPGA config) -I/O Connectors maximize"
- note removed: "ToDo: Fixup amp polarity and gains Calc all resistor Values"
- moved on the sheet: C1, C10, C11, C12, C13, C14, C15, C16, C17, C18, C19, C2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
